File: spliiter.kicad_pcb (KiCad board)
At the start: 2 copper layers, 78 parts, among them J1 JACK_TRS_6PINS, J2 JACK_TRS_6PINS, J3 JACK_TRS_6PINS, J4 JACK_TRS_6PINS, J5 JACK_TRS_6PINS, U1 NE5532, U2 NE5532, U3 NE5532, U4 NE5532, U5 NE5532

Commit message: pcb done
Parts:
- RV1, RV2, RV3, RV4: footprint Connect:PINHEAD1-3 -> Connect:PINHEAD1-6
- moved R6 214.2 mm to (79.0, 50.0), turned to 180 degrees
- moved R7 203.7 mm to (79.0, 67.0), turned to 180 degrees
- moved R10 202.4 mm to (79.0, 77.0), turned to 180 degrees
- moved R8 202.2 mm to (79.0, 70.0), turned to 180 degrees
- moved R5 201.1 mm to (79.0, 53.0), turned to 180 degrees
- moved C30 196.4 mm to (84.0, 60.0), turned to 270 degrees
- moved R11 196.0 mm to (79.0, 94.0), turned to 180 degrees
- moved R19 195.5 mm to (79.0, 148.0), turned to 180 degrees
- moved C35 192.0 mm to (84.0, 141.0), turned to 90 degrees
- moved R16 191.9 mm to (79.0, 124.0), turned to 180 degrees
- moved U3 190.1 mm to (79.0, 87.0), turned to 270 degrees
- moved RV2 189.2 mm to (72.0, 86.0), turned to 270 degrees
- moved R22 188.6 mm to (91.0, 64.0), turned to 270 degrees
- moved R21 188.1 mm to (91.0, 52.0), turned to 270 degrees
- moved C10 187.2 mm to (64.0, 95.0), turned to 90 degrees
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Routing:
- net VCC: track 0.00 -> 190.0 mm
- net Net-(RV1-Pad4): track 0.00 -> 187.1 mm
- net Net-(RV1-Pad1): track 0.00 -> 149.1 mm
- net GND: track 0.00 -> 86.8 mm, vias 0 -> 20
- net Net-(C2-Pad1): track 0.00 -> 25.6 mm, vias 0 -> 2
- net Net-(C1-Pad1): track 0.00 -> 23.6 mm, vias 0 -> 2
- net Net-(R22-Pad2): track 0.00 -> 18.3 mm
- net Net-(R15-Pad1): track 0.00 -> 17.5 mm
- net Net-(R19-Pad1): track 0.00 -> 17.5 mm
- net Net-(R11-Pad1): track 0.00 -> 17.5 mm
- net Net-(R17-Pad1): track 0.00 -> 16.3 mm
- net Net-(R23-Pad2): track 0.00 -> 16.3 mm
- net Net-(R13-Pad1): track 0.00 -> 16.3 mm
- net Net-(R21-Pad2): track 0.00 -> 16.3 mm
- net Net-(C9-Pad1): track 0.00 -> 9.23 mm
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- added copper zone on B.Cu, net GND
Other:
- board outline added: 57.5 x 127.5 mm
- net class Default: clearance 0.2 -> 0.3; trace_width 0.25 -> 0.3; via_dia 0.6 -> 0.7; via_drill 0.4 -> 0.5
- net class PWR added: clearance 0.5, trace_width 0.5, via_dia 0.7, via_drill 0.5
- rule trace_clearance: 0.2 -> 0.3
